Commit message: add robotiq_coupler link and joint

File: Universal_Robots_ROS2_Description/urdf/ur_workcell.urdf.xacro (robot description, xacro)
@@ -91,5 +91,32 @@
      <origin xyz="0 0 0" rpy="0 0 0" />          <!-- position robot in the world -->
    </xacro:ur_robot>
-   <xacro:if value="$(arg sim_gazebo)">
+  <!-- robotiq gripper link -->
+  <link name="$(arg prefix)robotiq_coupler">
+    <visual>
+      <geometry>
+        <mesh filename="package://robotiq_85_description/meshes/robotiq_85_coupler/robotiq_85_coupler.stl" />
+      </geometry>
+      <material name="flat_black">
+        <color rgba="0 0 0 1"/>
+      </material>
+    </visual>
+    <collision>
+      <geometry>
+        <mesh filename="package://robotiq_85_description/meshes/robotiq_85_coupler/robotiq_85_coupler.stl" />
+      </geometry>
+    </collision>
+    <inertial>
+      <origin xyz="2.073e-05   1.45286e-03  -1.1049e-03" rpy="0 0 0" />
+      <mass value="0.168" />
+      <inertia ixx="6.69695624e-05" ixy="5.21511788e-09" ixz="-2.74383009e-08"
+                  iyy="7.85088161e-05" iyz="5.41105193e-07" izz="1.41819717e-04"/>
+    </inertial>
+  </link>
+  <joint name="$(arg prefix)robotiq_coupler_joint" type="fixed">
+    <origin xyz="0 0 0.004" rpy="0 0 ${-pi/2.0}" />
+    <parent link="$(arg prefix)tool0"/>
+    <child link="$(arg prefix)robotiq_coupler"/>
+  </joint>
+  <xacro:if value="$(arg sim_gazebo)">
     <!-- Gazebo plugins -->
     <gazebo reference="world">

Commit message: add robotiq coupler

File: Universal_Robots_ROS2_Description/urdf/ur_workcell.urdf.xacro (robot description, xacro)
@@ -95,5 +95,5 @@
     <visual>
       <geometry>
-        <mesh filename="package://robotiq_85_description/meshes/robotiq_85_coupler/robotiq_85_coupler.stl" />
+        <mesh filename="package://robotiq_85_description/meshes/visual/kinova_robotiq_coupler.dae" />
       </geometry>
       <material name="flat_black">
@@ -103,5 +103,5 @@
     <collision>
       <geometry>
-        <mesh filename="package://robotiq_85_description/meshes/robotiq_85_coupler/robotiq_85_coupler.stl" />
+        <mesh filename="package://robotiq_85_description/meshes/collision/kinova_robotiq_coupler.stl" />
       </geometry>
     </collision>

Commit message: add epick end effector

File: Universal_Robots_ROS2_Description/urdf/ur_workcell.urdf.xacro (robot description, xacro)
@@ -7,4 +7,10 @@
    <!-- import lab table macro -->
    <xacro:include filename="$(find lab_table_description)/urdf/table_macro.xacro"/>
+   <!-- robotiq 85 2-finger gripper macro -->
+   <xacro:include filename="$(find robotiq_85_description)/urdf/robotiq_85_gripper.urdf.xacro" />
+   <!-- vg10 vacuum gripper macro -->
+   <xacro:include filename="$(find vg10_description)/urdf/vg10_macro.xacro" />
+   <!-- robotiq epick gripper macro -->
+   <xacro:include filename="$(find robotiq_epick_suction_gripper_description)/urdf/robotiq_epick_model.urdf.xacro" />
    <!-- possible 'ur_type' values: ur3, ur3e, ur5, ur5e, ur10, ur10e, ur16e -->
    <!-- the default value should raise an error in case this was called without defining the type -->
@@ -92,5 +98,5 @@
    </xacro:ur_robot>
   <!-- robotiq gripper link -->
-  <link name="$(arg prefix)robotiq_coupler">
+  <!-- <link name="$(arg prefix)robotiq_coupler">
     <visual>
       <geometry>
@@ -117,5 +123,9 @@
     <parent link="$(arg prefix)tool0"/>
     <child link="$(arg prefix)robotiq_coupler"/>
-  </joint>
+  </joint> -->
+  <!-- robotiq epick -->
+  <xacro:epick prefix="$(arg prefix)" parent="$(arg prefix)tool0" robot_name="$(arg prefix)epick">
+    <orgin xyz="0 0 0.011" rpy="0 0 ${pi}"/>
+  </xacro:epick>
   <xacro:if value="$(arg sim_gazebo)">
     <!-- Gazebo plugins -->
